File: ANN_Kicad.kicad_sch (KiCad schematic)
At the start: 70 parts, among them IC1 STM32F030F4P6, J1 Conn_01x02, J2 Conn_01x05, U1 Inverting Op Amps, U10 Comparator, U11 Buffer Op Amps, U2 Summing Op Amps, U3 Weights For N1, U4 Weights For N1, U5 Weights For N2, U6 Weights For N2, U7 Weights For N3, U8 Weights For N3

Commit message: sch: replace comparator with TLV7034, correct component values
Comparator LM339N (U10) -> PTLV7034PWR (U9, TI TLV7034 quad, TSSOP-14).
Rail-to-rail inputs (VCM = V- .. V+ +0.1 = 0..3.40 V at 3.3 V) cover the
0.198..3.0997 V sum swing and the 1.65 V reference with margin; internal
hysteresis (10 mV typ) and a push-pull output remove the chatter and the
missing-pull-up findings. Verified in sim/ -- see tb06, tb08, tb10.

Resistor and capacitor values: in each case the Value field was already
the design intent and the placed part was wrong. Because every part here
is an UltraLibrarian download whose symbol name IS the MPN
(CRCW0603100KFKEA = 100k), editing the Value field only relabels -- the
part ordered stays whatever the symbol is named. Each of these therefore
needed a symbol pointed at the correct MPN, not a retyped field:

  R4-R6    100k -> 3.3k   CRCW06033K30FKEA  recentres the LDR dividers on
                          ~141 lux (room light) instead of ~1.5 lux (near
                          dark), and caps ADC source impedance at 3.3k
  R34-R36  1k   -> 330    CRCW0603330RFKEA  ~3 mA, the current at which the
                          TLV7034's VOL is actually specified
  R33      100k -> 10k    RC0603FR-0710KL   NRST pull-up (IC1 pin 4)
  C3       100nF-> 10nF   CC0603KRX7R8BB103 VDDA decoupling (IC1 pin 5)
  C4       100nF-> 1uF    CC0603KRX7R8BB105 VDDA bulk

New libraries created for CRCW06033K30FKEA, CRCW0603330RFKEA and
CC0603KRX7R8BB105 (1uF 25V X7R -- same Yageo CC0603 series as the existing
103/104) and registered in the global tables. R33 reuses the project's
existing 10k rather than adding a second 10k MPN to the BOM; that symbol
has 12.7mm pin spacing against the old part's 10.16mm, so its wiring was
redrawn by hand.

Verified: kicad-cli netlist diff shows connectivity otherwise untouched
across every edit; ERC reports 0 violations.
Parts:
- removed C14: 100nF, 100nF:CAP_CC0603KRX7R8BB104_YAG-M, symbol 100nF:CC0603KRX7R8BB104
- removed D1: LED_LEFT, 151051RS11000:WL-TMRC_5MM, symbol WL-TMRC_5MM:WL-TMRC_5MM
- removed D2, D3: LED_CENTER, 151051RS11000:WL-TMRC_5MM, symbol WL-TMRC_5MM:WL-TMRC_5MM
- removed R30, R31, R32: 1k, CRCW06031K00FKEA:RESC1508X50N, symbol CRCW06031K00FKEA:CRCW06031K00FKEA
- removed U10: Comparator, LM339N:N14, symbol LM339N:LM339N
- added C15: 100nF, 100nF:CAP_CC0603KRX7R8BB104_YAG-M, symbol 100nF:CC0603KRX7R8BB104
- added D4, D5, D6: LED, 151051RS11000:WL-TMRC_5MM, symbol WL-TMRC_5MM:WL-TMRC_5MM
- added R34, R35, R36: 330, CRCW0603330RFKEA:RESC1508X50N, symbol CRCW0603330RFKEA:CRCW0603330RFKEA
- added U9: Comparator, ul_PTLV7034PWR:TSSOP_7034PWR_TEX-M, symbol ul_PTLV7034PWR:PTLV7034PWR
- C3: footprint 100nF:CAP_CC0603KRX7R8BB104_YAG-M -> 10nf_0603:CAP_CC0603KRX7R8BB103_YAG-M; symbol 100nF:CC0603KRX7R8BB104 -> 10nf_0603:CC0603KRX7R8BB103
- C4: footprint 100nF:CAP_CC0603KRX7R8BB104_YAG-M -> 1uF:CAP_CC0603KRX7R8BB105_YAG-M; symbol 100nF:CC0603KRX7R8BB104 -> 1uF:CC0603KRX7R8BB105
- R33: footprint CRCW0603100KFKEA:RESC1508X50N -> RC0603_YAG:RC0603N_YAG; symbol CRCW0603100KFKEA:CRCW0603100KFKEA -> RC0603:RC0603FR-0710KL
- R4, R5, R6: value 100k -> 3.3k; footprint CRCW0603100KFKEA:RESC1508X50N -> CRCW06033K30FKEA:RESC1508X50N; symbol CRCW0603100KFKEA:CRCW0603100KFKEA -> CRCW06033K30FKEA:CRCW06033K30FKEA
Connections:
- net +3.3V: now also C15.2, R34.2, R35.2, R36.2, U9.12 (+IN_D), U9.4 (VCC)
- net GND: now also C15.1, U9.11 (VEE), U9.13 (-IN_D)
- net N1_SUM: now also U9.3 (+IN_A)
- net N2_SUM: now also U9.5 (+IN_B)
- net N3_SUM: now also U9.10 (+IN_C)
- net V_REF_BUF: now also U9.2 (-IN_A), U9.6 (-IN_B), U9.9 (-IN_C)
- new net: D6.1, R36.1
- new net: D6.2, U9.7 (OUT_B)
- new net: D5.1, R35.1
- new net: D4.1, R34.1
- new net: D4.2, U9.1 (OUT_A)
- new net: D5.2, U9.8 (OUT_C)
- no-connect marks 8 -> 9
